File: alphabat_PCB.kicad_sch (KiCad schematic)
At the start: 14 parts

Commit message: ROWs n COLs
Parts:
- added A, B, C, D, E, ENT, F, G, H, I, J, K, L, M, N, O, P, Q, R, S, Space, T, U, V (x2), W, X, Y, Z: MX-NoLED, symbol MX_Alps_Hybrid:MX-NoLED
- added D? (x29): SOD-123, symbol Device:D_Small
- added J?: USB_C_Receptacle_USB2.0, symbol Connector:USB_C_Receptacle_USB2.0
Connections:
- new net: D?.2 (A), H.2 (ROW)
- new net: D?.2 (A), V.2 (ROW) (x2)
- new net: B.2 (ROW), D?.2 (A)
- new net: D?.2 (A), G.2 (ROW)
- new net: D?.2 (A), ENT.2 (ROW)
- new net: D?.2 (A), P.2 (ROW)
- new net: D?.2 (A), J.2 (ROW)
- new net: D.2 (ROW), D?.2 (A)
- new net: D?.2 (A), Space.2 (ROW)
- new net: D?.2 (A), I.2 (ROW)
- new net: D?.2 (A), N.2 (ROW)
- new net: D?.2 (A), O.2 (ROW)
- new net: D?.2 (A), F.2 (ROW)
- new net: D?.2 (A), W.2 (ROW)
- new net: D?.2 (A), Z.2 (ROW)
- new net: D?.2 (A), Q.2 (ROW)
- new net: D?.2 (A), S.2 (ROW)
- new net: D?.2 (A), E.2 (ROW)
- new net: D?.2 (A), U.2 (ROW)
- new net: D?.2 (A), X.2 (ROW)
- new net: D?.2 (A), K.2 (ROW)
- new net: J?.A1 (GND), J?.A12 (GND), J?.B1 (GND), J?.B12 (GND)
- new net: J?.A4 (VBUS), J?.A9 (VBUS), J?.B4 (VBUS), J?.B9 (VBUS)
- new net: D?.2 (A), L.2 (ROW)
- new net: D?.2 (A), M.2 (ROW)
- new net: D?.2 (A), R.2 (ROW)
- new net: D?.2 (A), T.2 (ROW)
- new net: D?.2 (A), Y.2 (ROW)
- new net: A.2 (ROW), D?.2 (A)
- new net: C.2 (ROW), D?.2 (A)
- new net COL0: A.1 (COL), Q.1 (COL), Z.1 (COL)
- new net COL1: S.1 (COL), W.1 (COL), X.1 (COL)
- new net COL2: C.1 (COL), D.1 (COL), E.1 (COL)
- new net COL3: F.1 (COL), R.1 (COL), V.1 (COL)
- new net COL4: B.1 (COL), G.1 (COL), T.1 (COL)
- new net COL5: H.1 (COL), Y.1 (COL)
- new net COL6: I.1 (COL), J.1 (COL), K.1 (COL), Space.1 (COL), U.1 (COL), V.1 (COL)
- new net COL7: L.1 (COL), N.1 (COL), O.1 (COL)
- new net COL8: ENT.1 (COL), M.1 (COL), P.1 (COL)
- new net ROW0: D?.1 (K), D?.1 (K), D?.1 (K), D?.1 (K), D?.1 (K), D?.1 (K), D?.1 (K), D?.1 (K), D?.1 (K), D?.1 (K)
- new net ROW1: D?.1 (K), D?.1 (K), D?.1 (K), D?.1 (K), D?.1 (K), D?.1 (K), D?.1 (K), D?.1 (K), D?.1 (K), D?.1 (K)
- new net ROW2: D?.1 (K), D?.1 (K), D?.1 (K), D?.1 (K), D?.1 (K), D?.1 (K), D?.1 (K), D?.1 (K), D?.1 (K)
Other:
- moved on the sheet: C?, R?, SW?, U?, Y?

Commit message: USB C
Parts:
- removed J?: USB_C_Receptacle_USB2.0, symbol Connector:USB_C_Receptacle_USB2.0
- added F?: 500m, symbol Device:Polyfuse_Small
- added R? (x2): 22, symbol Device:R_Small
- added R? (x2): 5.1k, symbol Device:R_Small
- added U?: PRTR5V0U2X, symbol random-keyboard-parts:PRTR5V0U2X
- added USB?: HRO-TYPE-C-31-M-12, symbol Type-C:HRO-TYPE-C-31-M-12
Connections:
- net +5V: now also F?.2
- net D+: now also R?.2
- net D-: now also R?.2
- net GND: now also R?.1, R?.2, U?.1 (GND), USB?.1 (GND), USB?.12 (GND), USB?.13 (SHIELD)
- new net: R?.1, U?.3 (IO2), USB?.5 (DN2), USB?.7 (DN1)
- new net: R?.1, U?.2 (IO1), USB?.6 (DP1), USB?.8 (DP2)
- new net: R?.2, USB?.10 (CC2)
- new net: R?.1, USB?.4 (CC1)
- new net VCC: F?.1, U?.4 (VCC), USB?.11 (VBUS), USB?.2 (VBUS)
- no-connect marks 0 -> 2
